File: DreamPad/DreamPad.kicad_pcb (KiCad board)
At the start: 2 copper layers, 75.8 x 93.2 mm, 25 parts, among them J1 OLED Display, SW1 SW_Push, SW10 SW_Push, SW11 SW_Push, SW13 RotaryEncoder_Switch, SW2 SW_Push, SW3 SW_Push, SW5 SW_Push, SW6 SW_Push, SW7 SW_Push, SW9 SW_Push, U1 MOUDLE-SEEEDUINO-XIAO

Commit message: Finalization and Readme
Parts:
- added H5: MountingHole, MountingHole:MountingHole_3.2mm_M3, F.Cu at (182.2, 110.2)
- moved H4 43.5 mm to (138.2, 132.8)
Connections:
- J1 pad 1: GND -> SDA
- J1 pad 2: Net-(J1-Pin_2) -> SCL
- J1 pad 3: SDA -> Net-(J1-Pin_3)
- J1 pad 4: SCL -> GND
- U1 pad 14: Net-(J1-Pin_2) -> Net-(J1-Pin_3)
Routing:
- net Net-(J1-Pin_2): track 66.3 -> 0.00 mm
- net Net-(J1-Pin_3): track 0.00 -> 65.2 mm
- net Net-(U1-PA5_A9_D9_MISO): track 129.7 -> 118.5 mm
- net SDA: track 103.8 -> 112.8 mm
- net Row 1: track 269.1 -> 261.9 mm
- net GND: track 130.3 -> 125.0 mm
- net SCL: track 93.9 -> 99.0 mm, vias 1 -> 2
Other:
- board size 75.8 x 93.2 mm -> 76 x 95.2 mm
